File: Carrier Board.brd (EAGLE design)
At the start: 90 x 38.6 mm, 67 parts, among them J1 S2B-PH-SM4-TB(LF)(SN), J2 S2B-PH-SM4-TB(LF)(SN), J3 BM04B-SRSS-TB(LF)(SN), J4 BM06B-SRSS-TB(LF)(SN), J5 BM06B-SRSS-TB(LF)(SN), J6 BM06B-SRSS-TB(LF)(SN), J7 BM04B-SRSS-TB(LF)(SN), J8 BM04B-SRSS-TB(LF)(SN), J9 BM04B-SRSS-TB(LF)(SN), P1 Particle Boron / Xenon / Argon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

Commit message: -Added logo -Production ready
Parts:
- removed U$2: (no value), SparkFun-Aesthetics:OSHW-LOGO-M
- moved FD2 82.0 mm to (84.3, 2.05), turned to 134.9 degrees
Other:
- board text added: "Designed by Charles McClelland"
- board text added: "Kumva RMS - Based on Carrier Board"
- board text added: "www.kumva.io"
- board text removed: "chip@seeinsights.com"
- board text removed: "v1.4- 7-22-20"

Commit message: Final_Production_Ready
Parts:
- moved FD2 82.6 mm to (1.69, 1.35)
Other:
- board text added: "Kumva IoT - Carrier Board designed"
- board text added: "by Charles McClelland, See Insights"
- board text removed: "Designed by Charles McClelland"
- board text removed: "Kumva RMS - Based on Carrier Board"
